File: PCB/BezelBud/BezelBud.kicad_sch (KiCad schematic)
At the start: 69 parts, among them J1 USB_C_Receptacle_USB2.0_16P, J2 Conn_01x05_Pin, SW1 SW_SPDT, SW2 SW_SPDT, SW3 SW_SPDT, SW4 SW_SPDT, SW5 SW_SPDT, SW6 SW_SPDT, SW7 SW_SPDT, SW8 SW_SPDT, SW9 SW_SPDT, U1 STM32G431CBT6, U2 USBLC6-2SC6, U3 LP5907MFX-3.3, U4 LP5907MFX-3.3, U5 PCM1861DBT, Y1 Crystal_GND24

Commit message: Updated PCB
Parts:
- added C31: 0.1uF, Capacitor_SMD:C_0603_1608Metric, symbol Device:C
- added R14: 1M, Resistor_SMD:R_0603_1608Metric, symbol Device:R
- C18: Rating X7R -> X5R
Connections:
- net GND: now also C31.2, R14.2; no longer J1.S1 (SHIELD)
- net G_A: now reaches D2.2 (A), R4.2
- net R_A: now reaches D1.2 (A), R3.2
- new net SHIELD: C31.1, J1.S1 (SHIELD), R14.1
- no-connect marks 29 -> 32
Other:
- moved on the sheet: R3, R4

Commit message: Added bleed resistor and cap to shield <> GND con
Parts:
- removed H1, H2, H3, H4: MountingHole, MountingHole:MountingHole_3.2mm_M3_Pad_Via, symbol Mechanical:MountingHole
- added H1, H2, H3, H4: MountingHole_Pad, MountingHole:MountingHole_3.2mm_M3_Pad_Via, symbol Mechanical:MountingHole_Pad
- renumbered C31 to C11, C11 to C12, C12 to C13, C13 to C14, C14 to C15, C15 to C16, C16 to C17, C17 to C18, C18 to C19, C19 to C20, C20 to C21, C21 to C22, C22 to C23, C23 to C24, C24 to C25, C25 to C26, C26 to C27, C27 to C28, C28 to C29, C29 to C30, C30 to C31, R2 to R1, R9 to R10, R10 to R11, R11 to R12, R12 to R13, R13 to R14, R1 to R2, R14 to R8, R8 to R9, SW2 to SW1, SW1 to SW2
Connections:
- net GND: now also H1.1, H2.1, H3.1, H4.1

Commit message: remapped int pin to avoid crossing
Connections:
- net INT: now also U1.25 (PB11); no longer U1.31 (PA9)
Other:
- note added: "AUDIO ADC"
- note added: "INPUT PWR + FILTER + 3V3/3V3A"
- note added: "MCU"
- note added: "MOUNTING"
- note removed: "Remove microphones for the board, leave solderig spot for wire. USB to be 90 degree flat"
- company: (none) -> Kay
- title: (none) -> Bevel Bud
- moved on the sheet: C1, C10, C11, C12, C13, C14, C15, C16, C17, C18, C19, C2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
