File: PCB/BezelBud/BezelBud.kicad_pcb (KiCad board)
At the start: 4 copper layers, 69 x 39 mm, 69 parts, among them J1 USB_C_Receptacle_USB2.0_16P, J2 Conn_01x05_Pin, SW1 SW_SPDT, SW2 SW_SPDT, SW3 SW_SPDT, SW4 SW_SPDT, SW5 SW_SPDT, SW6 SW_SPDT, SW7 SW_SPDT, SW8 SW_SPDT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

Commit message: Moved Led by switch, moved mute led and mute switch to closer pin
Parts:
- moved D1 46.3 mm to (118.6, 95.9), turned to 180 degrees
- moved R3 42.4 mm to (122.3, 91.4), turned to 180 degrees
- moved R1 1.26 mm to (138.6, 86.0)
- turned R4 to 180 degrees
Connections:
- U1 pad 39: unconnected-(U1-PA15-Pad39) -> /LED_LIVE
- U1 pad 40: unconnected-(U1-PB3-Pad40) -> /MUTE_SW
- U1 pad 42: /LED_LIVE -> unconnected-(U1-PB5-Pad42)
- U1 pad 43: /MUTE_SW -> unconnected-(U1-PB6-Pad43)
Routing:
- net /LED_LIVE: track 30.2 -> 46.0 mm
- net +3.3V: track 73.6 -> 81.0 mm
- net /R_A: track 1.75 -> 7.94 mm
- net /LED_BLINK: track 30.0 -> 25.7 mm
- net /SW_H: track 18.0 -> 16.7 mm
- net /G_A: track 1.75 -> 2.43 mm
- net GND: vias 85 -> 84
Other:
- board text removed: "ON"
